Commit message: v2 restarted as the extended Berkeley Humanoid Lite, built from BHL's own parts
The styled design is now what the BHL paper draws in its Fig. 5: the robot
brought to adult size with carbon-fibre tubes between its actuator modules,
the hip reordered to pitch/abduction/rotation, a dexterous hand.

tools/bhl_pieces.py cuts eleven printed parts out of BHL's published link
meshes (CC BY-SA 4.0): the actuator modules removed, the arms cut where a
tube takes over, the arm links straightened, the foot cradle raised 15 mm;
each piece carries its surface samples, hull and mass. tools/build_v2.py
places them on the 1.64 m skeleton with RobStride actuators in their cradles
by BHL's module classes (RS02 for the 5010s, RS06 for the shoulder's 6512,
an RS03 in the knee cradle, bored out, because 36 N·m did not hold the
crouch), tubes on printed socket flanges, BHL's 6803 yoke bearings, our hip
stack, torso and hands.

The shape pipeline gained a mesh shape: GLB pieces in the viewer, surface
samples and hulls in the audit, boxes in the URDF, additions-only STLs in
the parts builder. Audit clean (the straight-arm hip-roll coupling stays
documented); MuJoCo stands, crouches and takes 10 N·s with the RS02 ankles
at a servo stiffness above the pendulum's. aesthetic.html rewritten; the
AI Sapiens K1 study and skeleton are removed.

Co-Authored-By: Claude Fable 5.1 <noreply@anthropic.com>

File: assets/model/foh_v2_0.urdf (robot description, URDF)
Before this commit: robot foh_v2_0, 24 links, 23 joints
Links:
- removed link shoulder_roll_bracket_L
- removed link shoulder_roll_bracket_R
- removed link torso
- removed link upper_arm_yoke_L
- removed link upper_arm_yoke_R
- added link elbow_bracket_L, mass 0.4760; collision box size=0.06040 0.07350 0.07700; collision cylinder length=0.00300 radius=0.02200
- added link elbow_bracket_R, mass 0.4760; collision box size=0.06040 0.07350 0.07700; collision cylinder length=0.00300 radius=0.02200
- added link shoulder_bracket_L, mass 0.4880; collision box size=0.07750 0.07700 0.07200; collision cylinder length=0.00300 radius=0.02300
- added link shoulder_bracket_R, mass 0.4880; collision box size=0.07750 0.07700 0.07200; collision cylinder length=0.00300 radius=0.02300
- link ankle_block_L: mass 0.8860 -> 0.1750; geometry collision box size=0.05540 0.09900 0.10670; collision cylinder length=0.00300 radius=0.02200
- link ankle_block_R: mass 0.8860 -> 0.1750; geometry collision box size=0.05540 0.09900 0.10670; collision cylinder length=0.00300 radius=0.02200
- link foot_L: mass 0.2960 -> 0.8720; geometry collision box size=0.02800 0.00800 0.02000; collision box size=0.02800 0.00800 0.02000
- link foot_R: mass 0.2960 -> 0.8720; geometry collision box size=0.02800 0.00800 0.02000; collision box size=0.02800 0.00800 0.02000
- link forearm_L: mass 0.3110 -> 0.7570; geometry collision box size=0.05000 0.01400 0.00800; collision box size=0.05000 0.05000 0.00800
- link forearm_R: mass 0.3110 -> 0.7570; geometry collision box size=0.05000 0.01400 0.00800; collision box size=0.05000 0.05000 0.00800
- link hand_L: mass 0.4130 -> 0.4160; geometry collision box size=0.01400 0.02000 0.07500; collision box size=0.01400 0.02000 0.07500
- link hand_R: mass 0.4130 -> 0.4160; geometry collision box size=0.01400 0.02000 0.07500; collision box size=0.01400 0.02000 0.07500
- link pelvis: mass 2.3940 -> 11.7530; geometry collision box size=0.00300 0.14000 0.30000; collision box size=0.00300 0.33000 0.48000
- link shank_L: mass 1.3920 -> 0.8520; geometry collision box size=0.05300 0.08500 0.09400; collision box size=0.05300 0.10400 0.08650
- link shank_R: mass 1.3920 -> 0.8520; geometry collision box size=0.05300 0.08500 0.09400; collision box size=0.05300 0.10400 0.08650
- link thigh_L: mass 1.2620 -> 1.2890; geometry collision box size=0.06000 0.06000 0.00800; collision box size=0.08130 0.07700 0.10300
- link thigh_R: mass 1.2620 -> 1.2890; geometry collision box size=0.06000 0.06000 0.00800; collision box size=0.08130 0.07700 0.10300
- link upper_arm_L: mass 0.5460 -> 0.7500; geometry collision box size=0.03600 0.05000 0.00800; collision box size=0.05000 0.05000 0.00800
- link upper_arm_R: mass 0.5460 -> 0.7500; geometry collision box size=0.03600 0.05000 0.00800; collision box size=0.05000 0.05000 0.00800
Joints:
- removed joint waist_yaw
- joint ankle_pitch_L: limit lower=-0.7854 upper=0.7854 effort=60 velocity=20 -> lower=-0.7854 upper=0.7854 effort=17 velocity=20; origin xyz=0.00000 0.00025 -0.25750 rpy=0 0 0 -> xyz=0.00000 0.00000 -0.41500 rpy=0 0 0
- joint ankle_pitch_R: limit lower=-0.7854 upper=0.7854 effort=60 velocity=20 -> lower=-0.7854 upper=0.7854 effort=17 velocity=20; origin xyz=0.00000 -0.00025 -0.25750 rpy=0 0 0 -> xyz=0.00000 0.00000 -0.41500 rpy=0 0 0
- joint ankle_roll_L: limit lower=-0.4363 upper=0.4363 effort=36 velocity=20 -> lower=-0.4363 upper=0.4363 effort=17 velocity=20; origin xyz=-0.07100 -0.05200 -0.03000 rpy=0 0 0 -> xyz=0.04000 0.02500 -0.05000 rpy=0 0 0
- joint ankle_roll_R: limit lower=-0.4363 upper=0.4363 effort=36 velocity=20 -> lower=-0.4363 upper=0.4363 effort=17 velocity=20; origin xyz=-0.07100 0.05200 -0.03000 rpy=0 0 0 -> xyz=0.04000 -0.02500 -0.05000 rpy=0 0 0
- joint elbow_L: limit lower=-1.0472 upper=0.6981 effort=17 velocity=20 -> lower=0.0000 upper=1.7453 effort=17 velocity=20; origin xyz=0.00000 0.03300 -0.07050 rpy=0 0 0 -> xyz=0.00000 -0.02450 -0.04300 rpy=0 0 0; parent upper_arm_L -> elbow_bracket_L
- joint elbow_R: limit lower=-1.0472 upper=0.6981 effort=17 velocity=20 -> lower=0.0000 upper=1.7453 effort=17 velocity=20; origin xyz=0.00000 -0.03300 -0.07050 rpy=0 0 0 -> xyz=0.00000 0.02450 -0.04300 rpy=0 0 0; parent upper_arm_R -> elbow_bracket_R
- joint hip_pitch_L: origin xyz=0.00000 0.07400 0.71450 rpy=0 0 0 -> xyz=0.00000 0.07400 0.95000 rpy=0 0 0
- joint hip_pitch_R: origin xyz=0.00000 -0.07400 0.71450 rpy=0 0 0 -> xyz=0.00000 -0.07400 0.95000 rpy=0 0 0
- joint hip_roll_L: limit lower=-0.1396 upper=0.7854 effort=60 velocity=20 -> lower=-0.2094 upper=0.7854 effort=60 velocity=20; origin xyz=0.04600 0.06100 0.00000 rpy=0 0 0 -> xyz=0.04600 0.06600 0.00000 rpy=0 0 0
- joint hip_roll_R: limit lower=-0.1396 upper=0.7854 effort=60 velocity=20 -> lower=-0.2094 upper=0.7854 effort=60 velocity=20; origin xyz=0.04600 -0.06100 0.00000 rpy=0 0 0 -> xyz=0.04600 -0.06600 0.00000 rpy=0 0 0
- joint knee_L: origin xyz=0.00000 0.05175 -0.22050 rpy=0 0 0 -> xyz=-0.01150 -0.01000 -0.28350 rpy=0 0 0
- joint knee_R: origin xyz=0.00000 -0.05175 -0.22050 rpy=0 0 0 -> xyz=-0.01150 0.01000 -0.28350 rpy=0 0 0
- joint shoulder_pitch_L: child shoulder_roll_bracket_L -> shoulder_bracket_L; origin xyz=0.00000 0.08200 0.29650 rpy=0 0 0 -> xyz=0.00000 0.22000 1.42500 rpy=0 0 0; parent torso -> pelvis
- joint shoulder_pitch_R: child shoulder_roll_bracket_R -> shoulder_bracket_R; origin xyz=0.00000 -0.08200 0.29650 rpy=0 0 0 -> xyz=0.00000 -0.22000 1.42500 rpy=0 0 0; parent torso -> pelvis
- joint shoulder_roll_L: child upper_arm_yoke_L -> upper_arm_L; limit lower=0.0000 upper=2.6180 effort=36 velocity=20 -> lower=0.0000 upper=2.6180 effort=17 velocity=20; origin xyz=0.03600 0.07400 0.00000 rpy=0 0 0 -> xyz=0.02550 0.04300 0.00000 rpy=0 0 0; parent shoulder_roll_bracket_L -> shoulder_bracket_L
- joint shoulder_roll_R: child upper_arm_yoke_R -> upper_arm_R; limit lower=0.0000 upper=2.6180 effort=36 velocity=20 -> lower=0.0000 upper=2.6180 effort=17 velocity=20; origin xyz=0.03600 -0.07400 0.00000 rpy=0 0 0 -> xyz=0.02550 -0.04300 0.00000 rpy=0 0 0; parent shoulder_roll_bracket_R -> shoulder_bracket_R
- joint shoulder_yaw_L: child upper_arm_L -> elbow_bracket_L; limit lower=-0.2094 upper=1.5708 effort=17 velocity=20 -> lower=-1.5708 upper=1.5708 effort=17 velocity=20; origin xyz=-0.03600 0.00000 -0.11350 rpy=0 0 0 -> xyz=-0.00290 0.00000 -0.29700 rpy=0 0 0; parent upper_arm_yoke_L -> upper_arm_L
- joint shoulder_yaw_R: child upper_arm_R -> elbow_bracket_R; limit lower=-0.2094 upper=1.5708 effort=17 velocity=20 -> lower=-1.5708 upper=1.5708 effort=17 velocity=20; origin xyz=-0.03600 0.00000 -0.11350 rpy=0 0 0 -> xyz=-0.00290 0.00000 -0.29700 rpy=0 0 0; parent upper_arm_yoke_R -> upper_arm_R
- joint wrist_roll_L: axis 1 0 0 -> 0 0 1; limit lower=-3.1416 upper=3.1416 effort=5.5 velocity=20 -> lower=-3.1416 upper=3.1416 effort=17 velocity=20; origin xyz=0.10400 -0.03300 0.00000 rpy=0 0 0 -> xyz=0.00000 0.02960 -0.27000 rpy=0 0 0
- joint wrist_roll_R: axis -1 0 0 -> 0 0 -1; limit lower=-3.1416 upper=3.1416 effort=5.5 velocity=20 -> lower=-3.1416 upper=3.1416 effort=17 velocity=20; origin xyz=0.10400 0.03300 0.00000 rpy=0 0 0 -> xyz=0.00000 -0.02960 -0.27000 rpy=0 0 0

Commit message: v2: torso cage narrowed to BHL's proportion, shoulder actuators outside it
The 2020 cage is now 130 x 172 outside, as narrow as the mini PC allows
(BHL's is 140 x 160); the packs, computer, boards and power parts stack
vertically inside it, and the shoulder RS06s sit outside on a printed plate
and beam bolted to the side uprights, as BHL's modules do. Audit clean,
MuJoCo unchanged (stands, crouches, pushes to 10 N.s), 28 kg.

Co-Authored-By: Claude Fable 5.1 <noreply@anthropic.com>

File: assets/model/foh_v2_0.urdf (robot description, URDF)
Before this commit: robot foh_v2_0, 23 links, 22 joints
Links:
- link pelvis: mass 11.7530 -> 10.2640; geometry collision box size=0.00300 0.17200 0.48000; collision box size=0.00300 0.17200 0.48000
Joints:
- joint shoulder_pitch_L: origin xyz=0.00000 0.22000 1.42500 rpy=0 0 0 -> xyz=0.00000 0.19800 1.42500 rpy=0 0 0
- joint shoulder_pitch_R: origin xyz=0.00000 -0.22000 1.42500 rpy=0 0 0 -> xyz=0.00000 -0.19800 1.42500 rpy=0 0 0
