Commit message: v1 production design: BHL's extended configuration on RobStride, with its own page
tools/build_v1.py generates the production design: the paper's adult-sized
Fig. 5 layout (hip pitch/abduction/rotation stack on pelvis bars, one
carbon-fibre tube per thigh, shank, upper arm and forearm between printed
actuator cups, extrusion torso, dexterous hand) on RobStride RS04/03/06/02/05.
RS04 interface dimensioned from the RS04 manual; laser-cut aluminium plates;
polycarbonate covers; Amazing Hands. 1.64 m, 33 kg, 22 joints, core $6,325.

Screw lengths are now computed from ring thickness, counterbore and thread
depth with an engagement assertion (RS03/RS06 ring thickness corrected).
Collision audit, printable STLs (assets/print_v1), URDF and MuJoCo check all
run on it (--model v1); viewer, BOM and printing pages take ?model=v1;
production.html presents it; catalog entry and builder modules added.

Fixed in both designs: the elbow axis, whose positive direction bent the
forearm backward.

Co-Authored-By: Claude Fable 5.1 <noreply@anthropic.com>

File: assets/model/foh_v0_2.urdf (robot description, URDF)
Before this commit: robot foh_v0_2, 24 links, 23 joints
Joints:
- joint elbow_L: axis 0 1 0 -> 0 -1 0
- joint elbow_R: axis 0 1 0 -> 0 -1 0

Commit message: v2: shoulders through the cage side as BHL's, arms hung 10 deg abducted at zero
The shoulder RS06s now pass through the sides of the narrow cage between
the corner uprights (an outside plate with the ring, an inside plate between
the uprights), putting the shoulders 347 mm apart, BHL's 352. The hands clear
the hip stack because the arms hang 10 deg abducted at the zero pose, as
BHL's hang 15 deg: joints gained a fixed zero offset (zero_deg) that the
URDF, the audit and the viewer apply. Audit clean, MuJoCo unchanged.

Co-Authored-By: Claude Fable 5.1 <noreply@anthropic.com>

File: assets/model/foh_v0_2.urdf (robot description, URDF)
Before this commit: robot foh_v0_2, 24 links, 23 joints
Joints:
- joint ankle_pitch_L: origin xyz=0.00000 0.01625 -0.16300 rpy=0 0 0 -> xyz=0.00000 0.01625 -0.16300 rpy=0.00000 0.00000 0.00000
- joint ankle_pitch_R: origin xyz=0.00000 -0.01625 -0.16300 rpy=0 0 0 -> xyz=0.00000 -0.01625 -0.16300 rpy=0.00000 0.00000 0.00000
- joint ankle_roll_L: origin xyz=-0.06500 -0.05000 -0.03000 rpy=0 0 0 -> xyz=-0.06500 -0.05000 -0.03000 rpy=0.00000 0.00000 0.00000
- joint ankle_roll_R: origin xyz=-0.06500 0.05000 -0.03000 rpy=0 0 0 -> xyz=-0.06500 0.05000 -0.03000 rpy=-0.00000 0.00000 0.00000
- joint elbow_L: origin xyz=0.00000 0.03300 -0.09650 rpy=0 0 0 -> xyz=0.00000 0.03300 -0.09650 rpy=0.00000 -0.00000 0.00000
- joint elbow_R: origin xyz=0.00000 -0.03300 -0.09650 rpy=0 0 0 -> xyz=0.00000 -0.03300 -0.09650 rpy=0.00000 -0.00000 0.00000
- joint hip_pitch_L: origin xyz=0.00000 0.07400 0.46000 rpy=0 0 0 -> xyz=0.00000 0.07400 0.46000 rpy=0.00000 0.00000 0.00000
- joint hip_pitch_R: origin xyz=0.00000 -0.07400 0.46000 rpy=0 0 0 -> xyz=0.00000 -0.07400 0.46000 rpy=0.00000 0.00000 0.00000
- joint hip_roll_L: origin xyz=0.04400 0.05800 0.00000 rpy=0 0 0 -> xyz=0.04400 0.05800 0.00000 rpy=0.00000 0.00000 0.00000
- joint hip_roll_R: origin xyz=0.04400 -0.05800 0.00000 rpy=0 0 0 -> xyz=0.04400 -0.05800 0.00000 rpy=-0.00000 0.00000 0.00000
- joint hip_yaw_L: origin xyz=-0.04400 0.00000 -0.13450 rpy=0 0 0 -> xyz=-0.04400 0.00000 -0.13450 rpy=0.00000 0.00000 0.00000
- joint hip_yaw_R: origin xyz=-0.04400 0.00000 -0.13450 rpy=0 0 0 -> xyz=-0.04400 0.00000 -0.13450 rpy=0.00000 0.00000 -0.00000
- joint knee_L: origin xyz=0.00000 0.04975 -0.06250 rpy=0 0 0 -> xyz=0.00000 0.04975 -0.06250 rpy=0.00000 0.00000 0.00000
- joint knee_R: origin xyz=0.00000 -0.04975 -0.06250 rpy=0 0 0 -> xyz=0.00000 -0.04975 -0.06250 rpy=0.00000 0.00000 0.00000
- joint shoulder_pitch_L: origin xyz=0.00000 0.09900 0.35000 rpy=0 0 0 -> xyz=0.00000 0.09900 0.35000 rpy=0.00000 0.00000 0.00000
- joint shoulder_pitch_R: origin xyz=0.00000 -0.09900 0.35000 rpy=0 0 0 -> xyz=0.00000 -0.09900 0.35000 rpy=0.00000 0.00000 0.00000
- joint shoulder_roll_L: origin xyz=0.03800 0.13300 0.00000 rpy=0 0 0 -> xyz=0.03800 0.13300 0.00000 rpy=0.00000 0.00000 0.00000
- joint shoulder_roll_R: origin xyz=0.03800 -0.13300 0.00000 rpy=0 0 0 -> xyz=0.03800 -0.13300 0.00000 rpy=-0.00000 0.00000 0.00000
- joint shoulder_yaw_L: origin xyz=-0.03800 0.00000 -0.11350 rpy=0 0 0 -> xyz=-0.03800 0.00000 -0.11350 rpy=0.00000 0.00000 0.00000
- joint shoulder_yaw_R: origin xyz=-0.03800 0.00000 -0.11350 rpy=0 0 0 -> xyz=-0.03800 0.00000 -0.11350 rpy=0.00000 0.00000 -0.00000
- joint waist: origin xyz=0.00000 0.00000 0.59000 rpy=0 0 0 -> xyz=0.00000 0.00000 0.59000 rpy=0.00000 0.00000 0.00000
- joint wrist_roll_L: origin xyz=0.00000 -0.03300 -0.19300 rpy=0 0 0 -> xyz=0.00000 -0.03300 -0.19300 rpy=0.00000 0.00000 0.00000
- joint wrist_roll_R: origin xyz=0.00000 0.03300 -0.19300 rpy=0 0 0 -> xyz=0.00000 0.03300 -0.19300 rpy=0.00000 0.00000 -0.00000

File: assets/model/foh_v2_0.urdf (robot description, URDF)
Before this commit: robot foh_v2_0, 23 links, 22 joints
Links:
- link pelvis: mass 10.2640 -> 9.8720; geometry collision box size=0.00300 0.17200 0.48000; collision box size=0.00300 0.17200 0.48000
Joints:
- joint ankle_pitch_L: origin xyz=0.00000 0.00000 -0.41500 rpy=0 0 0 -> xyz=0.00000 0.00000 -0.41500 rpy=0.00000 0.00000 0.00000
- joint ankle_pitch_R: origin xyz=0.00000 0.00000 -0.41500 rpy=0 0 0 -> xyz=0.00000 0.00000 -0.41500 rpy=0.00000 0.00000 0.00000
- joint ankle_roll_L: origin xyz=0.04000 0.02500 -0.05000 rpy=0 0 0 -> xyz=0.04000 0.02500 -0.05000 rpy=0.00000 0.00000 0.00000
- joint ankle_roll_R: origin xyz=0.04000 -0.02500 -0.05000 rpy=0 0 0 -> xyz=0.04000 -0.02500 -0.05000 rpy=-0.00000 0.00000 0.00000
- joint elbow_L: origin xyz=0.00000 -0.02450 -0.04300 rpy=0 0 0 -> xyz=0.00000 -0.02450 -0.04300 rpy=0.00000 -0.00000 0.00000
- joint elbow_R: origin xyz=0.00000 0.02450 -0.04300 rpy=0 0 0 -> xyz=0.00000 0.02450 -0.04300 rpy=0.00000 -0.00000 0.00000
- joint hip_pitch_L: origin xyz=0.00000 0.07400 0.95000 rpy=0 0 0 -> xyz=0.00000 0.07400 0.95000 rpy=0.00000 0.00000 0.00000
- joint hip_pitch_R: origin xyz=0.00000 -0.07400 0.95000 rpy=0 0 0 -> xyz=0.00000 -0.07400 0.95000 rpy=0.00000 0.00000 0.00000
- joint hip_roll_L: origin xyz=0.04600 0.06600 0.00000 rpy=0 0 0 -> xyz=0.04600 0.06600 0.00000 rpy=0.00000 0.00000 0.00000
- joint hip_roll_R: origin xyz=0.04600 -0.06600 0.00000 rpy=0 0 0 -> xyz=0.04600 -0.06600 0.00000 rpy=-0.00000 0.00000 0.00000
- joint hip_yaw_L: origin xyz=-0.04600 0.00000 -0.13650 rpy=0 0 0 -> xyz=-0.04600 0.00000 -0.13650 rpy=0.00000 0.00000 0.00000
- joint hip_yaw_R: origin xyz=-0.04600 0.00000 -0.13650 rpy=0 0 0 -> xyz=-0.04600 0.00000 -0.13650 rpy=0.00000 0.00000 -0.00000
- joint knee_L: origin xyz=-0.01150 -0.01000 -0.28350 rpy=0 0 0 -> xyz=-0.01150 -0.01000 -0.28350 rpy=0.00000 0.00000 0.00000
- joint knee_R: origin xyz=-0.01150 0.01000 -0.28350 rpy=0 0 0 -> xyz=-0.01150 0.01000 -0.28350 rpy=0.00000 0.00000 0.00000
- joint shoulder_pitch_L: origin xyz=0.00000 0.19800 1.42500 rpy=0 0 0 -> xyz=0.00000 0.13050 1.42500 rpy=0.00000 0.00000 0.00000
- joint shoulder_pitch_R: origin xyz=0.00000 -0.19800 1.42500 rpy=0 0 0 -> xyz=0.00000 -0.13050 1.42500 rpy=0.00000 0.00000 0.00000
- joint shoulder_roll_L: origin xyz=0.02550 0.04300 0.00000 rpy=0 0 0 -> xyz=0.02550 0.04300 0.00000 rpy=0.17453 0.00000 0.00000
- joint shoulder_roll_R: origin xyz=0.02550 -0.04300 0.00000 rpy=0 0 0 -> xyz=0.02550 -0.04300 0.00000 rpy=-0.17453 0.00000 0.00000
- joint shoulder_yaw_L: origin xyz=-0.00290 0.00000 -0.29700 rpy=0 0 0 -> xyz=-0.00290 0.00000 -0.29700 rpy=0.00000 0.00000 0.00000
- joint shoulder_yaw_R: origin xyz=-0.00290 0.00000 -0.29700 rpy=0 0 0 -> xyz=-0.00290 0.00000 -0.29700 rpy=0.00000 0.00000 -0.00000
- joint wrist_roll_L: origin xyz=0.00000 0.02960 -0.27000 rpy=0 0 0 -> xyz=0.00000 0.02960 -0.27000 rpy=0.00000 0.00000 0.00000
- joint wrist_roll_R: origin xyz=0.00000 -0.02960 -0.27000 rpy=0 0 0 -> xyz=0.00000 -0.02960 -0.27000 rpy=0.00000 0.00000 -0.00000
